Commit message: rebuild everything

File: swarm_robot_ros_sim/swarm_robot_description/urdf/two_wheel_robot.urdf (robot description, URDF)
Before this commit: robot two_wheel_robot, 3 links, 2 joints
Links:
- added link lidar_link, mass 0.0005; collision box size=0.0254 0.0254 0.00154; visual box size=0.0254 0.0254 0.00054
Joints:
- added joint lidar_joint: type fixed, parent body_link, child lidar_link, origin xyz=0 0 0 rpy=0 0 0, axis 0 1 0

Commit message: update model

File: swarm_robot_ros_sim/swarm_robot_description/urdf/two_wheel_robot.urdf (robot description, URDF)
Before this commit: robot two_wheel_robot, 4 links, 3 joints
Links:
- link body_link: mass 0.03 -> 0.3
- link left_wheel: mass 0.002 -> 0.01
- link right_wheel: mass 0.002 -> 0.01
